File: sensors.kicad_sch (KiCad schematic)
At the start: 19 parts, among them CN2 SM04B-SRSS-TB (LF)(SN), CN3 SM04B-SRSS-TB (LF)(SN), U12 TMP75AIDR, U4 OPT3004DNPR, U8 MPU6500, U9 SN74AHCT1G125DBVR

Commit message: Added pull up / pull down on mode pin tps
Connections:
- net IMU_INT: now reaches U8.12 (INT)
- no-connect marks 24 -> 23
Changed lines of the file:
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@@
-	)
-	(no_connect
-		(at 73.66 107.95)
 	)
 	(no_connect
@@
 		(pts
 			(xy 245.11 41.91) (xy 245.11 43.18)
+		)
+		(stroke
+			(width 0)
+			(type default)
+		)
+	)
+	(wire
+		(pts
+			(xy 67.31 107.95) (xy 73.66 107.95)
 		)
 		(stroke
@@
 		)
 	)
+	(hierarchical_label "IMU_INT"
+		(shape output)
+		(at 67.31 107.95 180)
+		(effects
+			(font
+				(size 1.27 1.27)
+			)
+			(justify right)
+		)
+	)

Commit message: Finished placement , added few TP's
Other:
- moved on the sheet: C51
Changed lines of the file:
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@@
 	(symbol
 		(lib_id "easyeda2kicad:CC0603KRX7R9BB104")
-		(at 40.64 119.38 90)
+		(at 40.64 119.38 270)
+		(mirror x)
 		(unit 1)
 		(exclude_from_sim no)
@@
 		(dnp no)
 		(property "Reference" "C51"
-			(at 42.672 115.316 90)
+			(at 38.608 115.316 90)
 			(effects
 				(font
@@
 		)
 		(property "Value" "CC0603KRX7R9BB104"
-			(at 44.45 120.6499 90)
+			(at 36.83 120.6499 90)
 			(effects
 				(font
@@
 		)
 		(property "Footprint" "easyeda2kicad:C0603"
-			(at 48.26 119.38 0)
+			(at 33.02 119.38 0)
 			(effects
 				(font
@@
 		)
 		(property "Datasheet" "https://lcsc.com/product-detail/Multilayer-Ceramic-Capacitors-MLCC-SMD-SMT_100nF-104-10-50V_C14663.html"
-			(at 50.8 119.38 0)
+			(at 30.48 119.38 0)
 			(effects
 				(font
@@
 		)
 		(property "Description" "100nF"
-			(at 44.704 117.094 90)
+			(at 36.576 117.094 90)
 			(effects
 				(font
@@
 		)
 		(property "LCSC Part" "C14663"
-			(at 53.34 119.38 0)
+			(at 27.94 119.38 0)
 			(effects
 				(font
