File: stm32.kicad_pcb (KiCad board)
At the start: 4 copper layers, 50 x 100 mm, 166 parts, among them CN1 SM04B-SRSS-TB (LF)(SN), CN2 SM04B-SRSS-TB (LF)(SN), CN3 SM04B-SRSS-TB (LF)(SN), J1 PZ254V-11-03P_C2937625, J2 PZ254V-11-03P_C2937625, J3 B2B-PH-SM4-TB (LF)(SN), J5 PZ254V-11-03P_C2937625, P1 TYPE-C 16PIN 2MD(073), Q1 DMG2301L-7, SW1 JS102011JCQN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

Commit message: Fixed some drc errors
Routing:
- net +5VP: track 95.9 -> 110.0 mm, vias 9 -> 13

Commit message: Finished board ,now to production
Parts:
- added G***: LOGO, picture:lishay, B.Cu at (73.5, 39.8)
- added TP5: TestPoint, TestPoint:TestPoint_Pad_2.0x2.0mm, B.Cu at (86.9, 111.2)
- added TP6: TestPoint, TestPoint:TestPoint_Pad_2.0x2.0mm, B.Cu at (90.8, 111.4)
- added TP7: TestPoint, TestPoint:TestPoint_Pad_2.0x2.0mm, B.Cu at (89.4, 95.3)
- added TP8: TestPoint, TestPoint:TestPoint_Pad_2.0x2.0mm, B.Cu at (94.0, 95.3)
- renumbered + to TP3, - to TP4
Routing:
- net /stm32_page/SPI1_MOSI: track 68.8 -> 78.0 mm
- net GND: track 209.0 -> 217.4 mm
- net +5V: track 277.4 -> 285.3 mm, vias 20 -> 21
- net /stm32_page/SPI1_SCK: track 75.3 -> 78.1 mm
- net /stm32_page/IMU_INT: track 56.9 -> 59.2 mm
- net +3V3: track 404.4 -> 406.6 mm
- net /USB/USB_D-: track 24.2 -> 25.3 mm
- net /stm32_page/SPI1_MISO: track 77.2 -> 78.1 mm
Other:
- board text added: "+"
- board text added: "+3.3V"
- board text added: "+5V"
- board text added: "-"
- board text added: "GND"
- board text added: "I2C"
- board text added: "Light sens"
- board text added: "ON OFF"
- board text added: "PWM"
- board text added: "RX"
- board text added: "STAT2"
- board text added: "STM32 EVB"
- board text added: "TX"
- board text added: "Temp sns"
- board text added: "UART"
- board text added: "VCP"
- board text added: "אייל למפל לישי אבו"
