File: usb_power.kicad_sch (KiCad schematic)
At the start: 52 parts, among them CN1 SM04B-SRSS-TB (LF)(SN), J3 B2B-PH-SM4-TB (LF)(SN), P1 TYPE-C 16PIN 2MD(073), Q1 DMG2301L-7, SW1 JS102011JCQN, U13 CH340C_C7464026, U2 MCP73833T-AMI/MF, U3 TPS631000DRLR, U5 XC6206P332MR_C347376, U6 INA260AIPWR

Commit message: WIP routing still not finished
Parts:
- added C54: CC0603KRX7R9BB104, easyeda2kicad:C0603, symbol easyeda2kicad:CC0603KRX7R9BB104
Connections:
- net +5V: now also C136.2, U5.3 (VIN), U6.14 (IN-), U6.15 (IN-), U6.16 (IN-); no longer C1.2, C133.2, C134.2, C53.1, R1.2, U3.1 (VOUT), U6.1 (IN+), U6.10 (VS), U6.12 (VBUS), U6.2 (IN+), U6.3 (IN+)
- net GND: now also C54.2
- new net 5V_B4_INA: C1.2, C133.2, C134.2, C53.1, C54.1, R1.2, U3.1 (VOUT), U6.1 (IN+), U6.10 (VS), U6.12 (VBUS), U6.2 (IN+), U6.3 (IN+)
Other:
- moved on the sheet: TP3, TP4

Commit message: Finished board ,now to production
Parts:
- added TP5, TP6, TP7, TP8: TestPoint, TestPoint:TestPoint_Pad_2.0x2.0mm, symbol Connector:TestPoint
Connections:
- net +3V3: now also TP7.1
- net +5V: now also TP5.1
- net GND: now also TP6.1, TP8.1
